Commit message: [FIX] meshes path

File: a1.urdf (robot description, URDF)
Before this commit: robot robot, 18 links, 17 joints
Links:
- link LF_calf: geometry collision box size=0.2 0.016 0.016; visual mesh filename=package://meshes/a1/calf.stl scale=1 1 1
- link LF_hip: geometry collision cylinder length=0.04 radius=0.046; visual mesh filename=package://meshes/a1/hip.stl scale=1 1 1
- link LF_thigh: geometry collision box size=0.2 0.03 0.034; collision cylinder length=0.04 radius=0.041
- link LH_calf: geometry collision box size=0.2 0.016 0.016; visual mesh filename=package://meshes/a1/calf.stl scale=1 1 1
- link LH_hip: geometry collision cylinder length=0.04 radius=0.046; visual mesh filename=package://meshes/a1/hip.stl scale=1 1 1
- link LH_thigh: geometry collision box size=0.2 0.03 0.034; collision cylinder length=0.04 radius=0.041
- link RF_calf: geometry collision box size=0.2 0.016 0.016; visual mesh filename=package://meshes/a1/calf.stl scale=1 1 1
- link RF_hip: geometry collision cylinder length=0.04 radius=0.046; visual mesh filename=package://meshes/a1/hip.stl scale=1 1 1
- link RF_thigh: geometry collision box size=0.2 0.03 0.034; collision cylinder length=0.04 radius=0.041
- link RH_calf: geometry collision box size=0.2 0.016 0.016; visual mesh filename=package://meshes/a1/calf.stl scale=1 1 1
- link RH_hip: geometry collision cylinder length=0.04 radius=0.046; visual mesh filename=package://meshes/a1/hip.stl scale=1 1 1
- link RH_thigh: geometry collision box size=0.2 0.03 0.034; collision cylinder length=0.04 radius=0.041
- link base: geometry collision box size=0.267 0.194 0.114; visual mesh filename=package://meshes/a1/trunk.stl scale=1 1 1

File: go1.urdf (robot description, URDF)
Before this commit: robot robot, 18 links, 17 joints
Links:
- link LF_calf: geometry collision box size=0.213 0.016 0.016; visual mesh filename=package://meshes/go1/calf.stl scale=1 1 1
- link LF_hip: geometry collision cylinder length=0.04 radius=0.046; visual mesh filename=package://meshes/go1/hip.stl scale=1 1 1
- link LF_thigh: geometry collision box size=0.213 0.0245 0.034; visual mesh filename=package://meshes/go1/thigh.stl scale=1 1 1
- link LH_calf: geometry collision box size=0.213 0.016 0.016; visual mesh filename=package://meshes/go1/calf.stl scale=1 1 1
- link LH_hip: geometry collision cylinder length=0.04 radius=0.046; visual mesh filename=package://meshes/go1/hip.stl scale=1 1 1
- link LH_thigh: geometry collision box size=0.213 0.0245 0.034; visual mesh filename=package://meshes/go1/thigh.stl scale=1 1 1
- link RF_calf: geometry collision box size=0.213 0.016 0.016; visual mesh filename=package://meshes/go1/calf.stl scale=1 1 1
- link RF_hip: geometry collision cylinder length=0.04 radius=0.046; visual mesh filename=package://meshes/go1/hip.stl scale=1 1 1
- link RF_thigh: geometry collision box size=0.213 0.0245 0.034; visual mesh filename=package://meshes/go1/thigh_mirror.stl scale=1 1 1
- link RH_calf: geometry collision box size=0.213 0.016 0.016; visual mesh filename=package://meshes/go1/calf.stl scale=1 1 1
- link RH_hip: geometry collision cylinder length=0.04 radius=0.046; visual mesh filename=package://meshes/go1/hip.stl scale=1 1 1
- link RH_thigh: geometry collision box size=0.213 0.0245 0.034; visual mesh filename=package://meshes/go1/thigh_mirror.stl scale=1 1 1
- link base: geometry collision box size=0.3762 0.0935 0.114; visual mesh filename=package://meshes/go1/trunk.stl scale=1 1 1

File: go1_floating_base.urdf (robot description, URDF)
Before this commit: robot go1, 36 links, 35 joints
Links:
- link lf_hip: geometry collision cylinder length=0.04 radius=0.046; visual mesh filename=package://meshes/go1_floating_base/hip.stl scale=1 1 1
- link lf_lowerleg: geometry collision box size=0.213 0.016 0.016; visual mesh filename=package://meshes/go1_floating_base/lowerleg.stl scale=1 1 1
- link lf_upperleg: geometry collision box size=0.213 0.0245 0.034; visual mesh filename=package://meshes/go1_floating_base/upperleg.stl scale=1 1 1
- link lh_hip: geometry collision cylinder length=0.04 radius=0.046; visual mesh filename=package://meshes/go1_floating_base/hip.stl scale=1 1 1
- link lh_lowerleg: geometry collision box size=0.213 0.016 0.016; visual mesh filename=package://meshes/go1_floating_base/lowerleg.stl scale=1 1 1
- link lh_upperleg: geometry collision box size=0.213 0.0245 0.034; visual mesh filename=package://meshes/go1_floating_base/upperleg.stl scale=1 1 1
- link rf_hip: geometry collision cylinder length=0.04 radius=0.046; visual mesh filename=package://meshes/go1_floating_base/hip.stl scale=1 1 1
- link rf_lowerleg: geometry collision box size=0.213 0.016 0.016; visual mesh filename=package://meshes/go1_floating_base/lowerleg.stl scale=1 1 1
- link rf_upperleg: geometry collision box size=0.213 0.0245 0.034; visual mesh filename=package://meshes/go1_floating_base/upperleg_mirror.stl scale=1 1 1
- link rh_hip: geometry collision cylinder length=0.04 radius=0.046; visual mesh filename=package://meshes/go1_floating_base/hip.stl scale=1 1 1
- link rh_lowerleg: geometry collision box size=0.213 0.016 0.016; visual mesh filename=package://meshes/go1_floating_base/lowerleg.stl scale=1 1 1
- link rh_upperleg: geometry collision box size=0.213 0.0245 0.034; visual mesh filename=package://meshes/go1_floating_base/upperleg_mirror.stl scale=1 1 1
- link trunk: geometry collision box size=0.3762 0.0935 0.114; visual mesh filename=package://meshes/go1_floating_base/trunk.stl scale=1 1 1
